File: kicad_files/Bare ESP8266/RatGDO-OpenSource-Bare-ESP8266.kicad_sch (KiCad schematic)
At the start: 20 parts, among them J1 Screw_Terminal_01x03, J2 Screw_Terminal_01x03, J3 Screw_Terminal_01x03, J4 Conn_01x04, J5 Screw_Terminal_01x02, J6 Conn_01x02, Q1 2N7002, Q2 AO3400A, SW1 SW_Push, U1 ESP-12F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

Commit message: Missed Silkscreening for programming header
Connections:
- net +12V: no longer U2.2 (-IN)
- net +3.3V: now also J4.3 (Pin_3)
- net GND: now also U2.2 (-IN), U2.4 (-OUT)
- net at R5.1, SW1.2, U1.18 (GPIO0): no longer J4.3 (Pin_3)
- net at J5.2 (+3.3V), J6.2 (Pin_2), U2.3 (+OUT): no longer U2.4 (-OUT)
Changed lines of the file:
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@@
   (junction (at 158.75 90.17) (diameter 0) (color 0 0 0 0)
   )
+  (junction (at 83.82 54.61) (diameter 0) (color 0 0 0 0)
+  )
   (junction (at 92.71 54.61) (diameter 0) (color 0 0 0 0)
   )
@@
   (junction (at 62.23 54.61) (diameter 0) (color 0 0 0 0)
   )
-  (junction (at 92.71 52.07) (diameter 0) (color 0 0 0 0)
-  )
   (junction (at 105.41 52.07) (diameter 0) (color 0 0 0 0)
   )
   (junction (at 158.75 87.63) (diameter 0) (color 0 0 0 0)
   )
-  (junction (at 77.47 38.1) (diameter 0) (color 0 0 0 0)
-  )
   (junction (at 128.27 105.41) (diameter 0) (color 0 0 0 0)
   )
@@
   (junction (at 143.51 90.17) (diameter 0) (color 0 0 0 0)
   )
-  (junction (at 31.75 38.1) (diameter 0) (color 0 0 0 0)
-  )
   (wire (pts (xy 58.42 69.85) (xy 58.42 68.58))
     (stroke (width 0) (type default))
@@
     (stroke (width 0) (type default))
   )
-  (wire (pts (xy 31.75 38.1) (xy 31.75 48.26))
+  (wire (pts (xy 31.75 31.75) (xy 31.75 48.26))
     (stroke (width 0) (type default))
   )
@@
     (stroke (width 0) (type default))
   )
-  (wire (pts (xy 62.23 38.1) (xy 77.47 38.1))
-    (stroke (width 0) (type default))
-  )
   (wire (pts (xy 125.73 66.04) (xy 121.92 66.04))
     (stroke (width 0) (type default))
@@
     (stroke (width 0) (type default))
   )
-  (wire (pts (xy 77.47 38.1) (xy 77.47 40.64))
+  (wire (pts (xy 77.47 31.75) (xy 77.47 40.64))
     (stroke (width 0) (type default))
   )
@@
     (stroke (width 0) (type default))
   )
+  (wire (pts (xy 83.82 48.26) (xy 83.82 54.61))
+    (stroke (width 0) (type default))
+  )
   (wire (pts (xy 158.75 90.17) (xy 181.61 90.17))
     (stroke (width 0) (type default))
@@
     (stroke (width 0) (type default))
   )
+  (wire (pts (xy 90.17 46.99) (xy 90.17 48.26))
+    (stroke (width 0) (type default))
+  )
   (wire (pts (xy 105.41 115.57) (xy 105.41 113.03))
     (stroke (width 0) (type default))
@@
     (stroke (width 0) (type default))
   )
+  (wire (pts (xy 90.17 48.26) (xy 83.82 48.26))
+    (stroke (width 0) (type default))
+  )
   (wire (pts (xy 113.03 69.85) (xy 105.41 69.85))
     (stroke (width 0) (type default))
@@
     (stroke (width 0) (type default))
   )
-  (wire (pts (xy 31.75 31.75) (xy 31.75 38.1))
+  (wire (pts (xy 62.23 38.1) (xy 63.5 38.1))
     (stroke (width 0) (type default))
   )
@@
     (stroke (width 0) (type default))
   )
-  (wire (pts (xy 44.45 38.1) (xy 31.75 38.1))
-    (stroke (width 0) (type default))
-  )
   (wire (pts (xy 121.92 66.04) (xy 121.92 74.93))
     (stroke (width 0) (type default))
@@
     (stroke (width 0) (type default))
   )
-  (wire (pts (xy 92.71 48.26) (xy 92.71 52.07))
-    (stroke (width 0) (type default))
-  )
-  (wire (pts (xy 77.47 31.75) (xy 77.47 38.1))
+  (wire (pts (xy 43.18 38.1) (xy 44.45 38.1))
     (stroke (width 0) (type default))
   )
@@
     (stroke (width 0) (type default))
   )
-  (wire (pts (xy 77.47 54.61) (xy 85.09 54.61))
+  (wire (pts (xy 77.47 54.61) (xy 83.82 54.61))
+    (stroke (width 0) (type default))
+  )
+  (wire (pts (xy 83.82 54.61) (xy 85.09 54.61))
     (stroke (width 0) (type default))
   )
@@
     (stroke (width 0) (type default))
   )
-  (wire (pts (xy 90.17 48.26) (xy 92.71 48.26))
-    (stroke (width 0) (type default))
-  )
   (wire (pts (xy 105.41 115.57) (xy 105.41 116.84))
     (stroke (width 0) (type default))
   )
   (wire (pts (xy 102.87 46.99) (xy 102.87 105.41))
-    (stroke (width 0) (type default))
-  )
-  (wire (pts (xy 90.17 46.99) (xy 90.17 48.26))
     (stroke (width 0) (type default))
   )
@@
     )
   )
+  (symbol (lib_id "power:GND") (at 43.18 38.1 270) (unit 1)
+    (in_bom yes) (on_board yes) (dnp no) (fields_autoplaced)
+    (property "Reference" "#PWR04" (at 36.83 38.1 0)
+      (effects (font (size 1.27 1.27)) hide)
+    )
+    (property "Value" "GND" (at 39.37 38.1 90)
+      (effects (font (size 1.27 1.27)) (justify right))
+    )
+    (property "Footprint" "" (at 43.18 38.1 0)
+      (effects (font (size 1.27 1.27)) hide)
+    )
+    (property "Datasheet" "" (at 43.18 38.1 0)
+      (effects (font (size 1.27 1.27)) hide)
+    )
+    (pin "1")
+    (instances
+      (project "RatGDO-OpenSource-Bare-ESP8266"
+        (path "/d526daf5-1a87-4c4a-b8db-6120ccadc008"
+          (reference "#PWR04") (unit 1)
+        )
+      )
+    )
+  )
   (symbol (lib_id "Device:R") (at 105.41 59.69 0) (unit 1)
     (in_bom yes) (on_board yes) (dnp no) (fields_autoplaced)
@@
         )
       )
+    )
+  )
+  (symbol (lib_id "power:GND") (at 63.5 38.1 90) (unit 1)
+    (in_bom yes) (on_board yes) (dnp no) (fields_autoplaced)
+    (property "Reference" "#PWR05" (at 69.85 38.1 0)
+      (effects (font (size 1.27 1.27)) hide)
+    )
+    (property "Value" "GND" (at 67.31 38.1 90)
+      (effects (font (size 1.27 1.27)) (justify right))
+    )
+    (property "Footprint" "" (at 63.5 38.1 0)
+      (effects (font (size 1.27 1.27)) hide)
+    )
+    (property "Datasheet" "" (at 63.5 38.1 0)
+      (effects (font (size 1.27 1.27)) hide)
+    )
+    (pin "1")
+    (instances
+      (project "RatGDO-OpenSource-Bare-ESP8266"
+        (path "/d526daf5-1a87-4c4a-b8db-6120ccadc008"
+          (reference "#PWR05") (unit 1)
+        )
+      )
